Commit message: 2024

File: rm_gimbal_description/urdf/rm_gimbal.urdf.xacro (robot description, xacro)
@@ -5,8 +5,13 @@
   <xacro:arg name="rpy" default="0 0 0" />
   <link name="odom" />
+  <link name="gimbal"/>
+  <joint name="gimbal_joint" type="floating">
+    <parent link="odom" />
+    <child link="gimbal" />
+  </joint>
   <link name="odom_link_first" />
   <joint name="odom_joint_first" type="fixed">
     <origin xyz="0 0.123 -0.140" rpy="$(arg rpy)" />
-    <parent link="odom" />
+    <parent link="gimbal" />
     <child link="odom_link_first" />
     <axis xyz="0 0 0" />
@@ -33,5 +38,5 @@
   <joint name="odom_joint_second" type="fixed">
     <origin xyz="0 -0.123 -0.140" rpy="$(arg rpy)" />
-    <parent link="odom" />
+    <parent link="gimbal" />
     <child link="odom_link_second" />
     <axis xyz="0 0 0" />

Commit message: 2024

File: rm_gimbal_description/urdf/rm_gimbal.urdf.xacro (robot description, xacro)
@@ -6,5 +6,5 @@
   <link name="odom" />
   <link name="gimbal"/>
-  <joint name="gimbal_joint" type="floating">
+  <joint name="gimbal_joint" type="fixed">
     <parent link="odom" />
     <child link="gimbal" />
@@ -18,5 +18,5 @@
   </joint>
   <link name="gimbal_link_first" />
-  <joint name="gimbal_joint_first" type="floating">
+  <joint name="gimbal_joint_first" type="fixed">
     <parent link="odom_link_first" />
     <child link="gimbal_link_first" />
@@ -43,5 +43,5 @@
   </joint>
   <link name="gimbal_link_second" />
-  <joint name="gimbal_joint_second" type="floating">
+  <joint name="gimbal_joint_second" type="fixed">
     <parent link="odom_link_second" />
     <child link="gimbal_link_second" />
